Commit message: Versión del robot ampliado

File: src/ros2_control/ros2_control_demo_description/r6bot/urdf/r6bot_description.urdf.xacro (robot description, xacro)
@@ -55,12 +55,13 @@
   <link name="ft_frame"/>
   <link name="tool0"/>
-  <!-- base_joint fixes base_link to the environment -->
-  <joint name="base_joint" type="fixed">
-    <parent link="world"/>
-    <child link="base_link"/>
-    <origin xyz="0 0 0" rpy="0 0 0"/>
-    <axis xyz="0 0 1"/>
-  </joint>
+  <link name="world"/>
   <!-- joints - main serial chain -->
+  <joint name="base_slider_joint" type="prismatic">
+  <parent link="world" />
+  <child link="base_link" />
+  <origin xyz="0 0 0" rpy="0 0 0" />
+  <axis xyz="1 0 0" />
+  <limit effort="1000.0" lower="-1.0" upper="1.0" velocity="0.5" />
+</joint>
   <joint name="joint_1" type="revolute">
     <parent link="base_link"/>

File: src/ros2_control/ros2_control_demo_example_7/description/ros2_control/r6bot.ros2_control.xacro (robot description, xacro)
@@ -6,4 +6,18 @@
         <plugin>ros2_control_demo_example_7/RobotSystem</plugin>
       </hardware>
+      <joint name="base_slider_joint">
+        <command_interface name="position">
+          <param name="min">-1.0</param>
+          <param name="max">1.0</param>
+        </command_interface>
+        <command_interface name="velocity">
+          <param name="min">-3.15</param>
+          <param name="max">3.15</param>
+        </command_interface>
+        <state_interface name="position">
+          <param name="initial_value">0.0</param>
+        </state_interface>
+        <state_interface name="velocity"/>
+        </joint>
       <joint name="joint_1">
         <command_interface name="position">

File: src/ros2_control_inicial/ros2_control_demo_description/r6bot/urdf/r6bot_description.urdf.xacro (robot description, xacro)
@@ -55,13 +55,12 @@
   <link name="ft_frame"/>
   <link name="tool0"/>
-  <link name="world"/>
+  <!-- base_joint fixes base_link to the environment -->
+  <joint name="base_joint" type="fixed">
+    <parent link="world"/>
+    <child link="base_link"/>
+    <origin xyz="0 0 0" rpy="0 0 0"/>
+    <axis xyz="0 0 1"/>
+  </joint>
   <!-- joints - main serial chain -->
-  <joint name="base_slider_joint" type="prismatic">
-  <parent link="world" />
-  <child link="base_link" />
-  <origin xyz="0 0 0" rpy="0 0 0" />
-  <axis xyz="1 0 0" />
-  <limit effort="1000.0" lower="-1.0" upper="1.0" velocity="0.5" />
-</joint>
   <joint name="joint_1" type="revolute">
     <parent link="base_link"/>

File: src/ros2_control_inicial/ros2_control_demo_example_7/description/ros2_control/r6bot.ros2_control.xacro (robot description, xacro)
@@ -6,18 +6,4 @@
         <plugin>ros2_control_demo_example_7/RobotSystem</plugin>
       </hardware>
-      <joint name="base_slider_joint">
-        <command_interface name="position">
-          <param name="min">-1.0</param>
-          <param name="max">1.0</param>
-        </command_interface>
-        <command_interface name="velocity">
-          <param name="min">-3.15</param>
-          <param name="max">3.15</param>
-        </command_interface>
-        <state_interface name="position">
-          <param name="initial_value">0.0</param>
-        </state_interface>
-        <state_interface name="velocity"/>
-        </joint>
       <joint name="joint_1">
         <command_interface name="position">

Commit message: Versión del robot ampliado

File: src/ros2_control/ros2_control_demo_description/r6bot/urdf/r6bot_description.urdf.xacro (robot description, xacro)
@@ -55,5 +55,4 @@
   <link name="ft_frame"/>
   <link name="tool0"/>
-  <link name="world"/>
   <!-- joints - main serial chain -->
   <joint name="base_slider_joint" type="prismatic">
@@ -63,5 +62,6 @@
   <axis xyz="1 0 0" />
   <limit effort="1000.0" lower="-1.0" upper="1.0" velocity="0.5" />
-</joint>
+  </joint>
+  <link name="world"/>
   <joint name="joint_1" type="revolute">
     <parent link="base_link"/>

File: src/ros2_control/ros2_control_demo_example_7/description/ros2_control/r6bot.ros2_control.xacro (robot description, xacro)
@@ -9,9 +9,5 @@
         <command_interface name="position">
           <param name="min">-1.0</param>
-          <param name="max">1.0</param>
-        </command_interface>
-        <command_interface name="velocity">
-          <param name="min">-3.15</param>
-          <param name="max">3.15</param>
+           <param name="max">1.0</param>
         </command_interface>
         <state_interface name="position">
@@ -19,5 +15,5 @@
         </state_interface>
         <state_interface name="velocity"/>
-        </joint>
+      </joint>
       <joint name="joint_1">
         <command_interface name="position">

Commit message: Versión modificada del robot

File: src/ros2_control/ros2_control_demo_description/r6bot/urdf/r6bot_description.urdf.xacro (robot description, xacro)
@@ -63,5 +63,5 @@
   <limit effort="1000.0" lower="-1.0" upper="1.0" velocity="0.5" />
   </joint>
-  <link name="world"/>
+  <!--<link name="world"/> -->
   <joint name="joint_1" type="revolute">
     <parent link="base_link"/>
